Commit message: add moveit

File: bentley_description/urdf/base_arm.xacro (robot description, xacro)
@@ -87,5 +87,5 @@
    <visual>
       <geometry>
-        <mesh filename="package://r1/meshes/gizmo_lift.stl" scale="${M_SCALE} ${M_SCALE} ${M_SCALE}"/>
+        <mesh filename="package://bentley/meshes/gizmo_lift.stl" scale="${M_SCALE} ${M_SCALE} ${M_SCALE}"/>
       </geometry>
          <xacro:yellow2/>
@@ -96,5 +96,5 @@
         <origin rpy="-1.57 0 0" xyz=" 0 0 0"/>
         <geometry>
-          <mesh filename="package://r1/meshes/gizmo_lift.stl" scale="${M_SCALE} ${M_SCALE} ${M_SCALE}"/>
+          <mesh filename="package://bentley/meshes/gizmo_lift.stl" scale="${M_SCALE} ${M_SCALE} ${M_SCALE}"/>
           </geometry>
       </collision>
@@ -120,5 +120,5 @@
    <visual>
       <geometry>
-        <mesh filename="package://r1/meshes/gizmo_lift.stl" scale="${M_SCALE} ${M_SCALE} ${M_SCALE}"/>
+        <mesh filename="package://bentley/meshes/gizmo_lift.stl" scale="${M_SCALE} ${M_SCALE} ${M_SCALE}"/>
       </geometry>
          <xacro:yellow2/>
@@ -129,5 +129,5 @@
         <origin rpy="1.57 0 0" xyz=" 0 0 0"/>
         <geometry>
-          <mesh filename="package://r1/meshes/gizmo_lift.stl" scale="${M_SCALE} ${M_SCALE} ${M_SCALE}"/>
+          <mesh filename="package://bentley/meshes/gizmo_lift.stl" scale="${M_SCALE} ${M_SCALE} ${M_SCALE}"/>
           </geometry>
       </collision>
